File: Button MIDI Controller.kicad_pcb (KiCad board)
At the start: 2 copper layers, 248.1 x 248.1 mm, 290 parts, among them J1 SWD, J2 USB_C_Receptacle_USB2.0_16P, U1 RP2040, U2 W25Q16JVZPIQ, U3 USBLC6-2SC6, U4 XC6206PxxxMR, Y1 X322512MSB4SI

Commit message: updates
Parts:
- removed D200: WS2812B-2020, LED_SMD:LED_WS2812B-2020_PLCC4_2.0x2.0mm
- added D65: WS2812B-2020, LED_SMD:LED_WS2812B-2020_PLCC4_2.0x2.0mm-notext, F.Cu at (-280.4, -312.7)
- added D66: WS2812B-2020, LED_SMD:LED_WS2812B-2020_PLCC4_2.0x2.0mm-notext, F.Cu at (-250.1, -312.7)
- added D67: WS2812B-2020, LED_SMD:LED_WS2812B-2020_PLCC4_2.0x2.0mm-notext, F.Cu at (-219.8, -312.7)
- added D68: WS2812B-2020, LED_SMD:LED_WS2812B-2020_PLCC4_2.0x2.0mm-notext, F.Cu at (-189.5, -312.7)
- added D69: WS2812B-2020, LED_SMD:LED_WS2812B-2020_PLCC4_2.0x2.0mm-notext, F.Cu at (-159.2, -312.7)
- added D70: WS2812B-2020, LED_SMD:LED_WS2812B-2020_PLCC4_2.0x2.0mm-notext, F.Cu at (-128.9, -312.7)
- added D71: WS2812B-2020, LED_SMD:LED_WS2812B-2020_PLCC4_2.0x2.0mm-notext, F.Cu at (-98.6, -312.7)
- added D72: WS2812B-2020, LED_SMD:LED_WS2812B-2020_PLCC4_2.0x2.0mm-notext, F.Cu at (-68.3, -312.7)
- added S1: TS11-674-120-BK-100-RA-D, TS11-674-120-BK-100-RA-D:SW_TS11-674-120-BK-100-RA-D, F.Cu at (-279.5, -289.1)
- added S2: TS11-674-120-BK-100-RA-D, TS11-674-120-BK-100-RA-D:SW_TS11-674-120-BK-100-RA-D, F.Cu at (-279.5, -258.9)
- added S3: TS11-674-120-BK-100-RA-D, TS11-674-120-BK-100-RA-D:SW_TS11-674-120-BK-100-RA-D, F.Cu at (-279.5, -228.6)
- added S4: TS11-674-120-BK-100-RA-D, TS11-674-120-BK-100-RA-D:SW_TS11-674-120-BK-100-RA-D, F.Cu at (-279.5, -198.2)
- added S5: TS11-674-120-BK-100-RA-D, TS11-674-120-BK-100-RA-D:SW_TS11-674-120-BK-100-RA-D, F.Cu at (-279.5, -167.9)
- added S6: TS11-674-120-BK-100-RA-D, TS11-674-120-BK-100-RA-D:SW_TS11-674-120-BK-100-RA-D, F.Cu at (-279.5, -137.7)
- added S7: TS11-674-120-BK-100-RA-D, TS11-674-120-BK-100-RA-D:SW_TS11-674-120-BK-100-RA-D, F.Cu at (-279.5, -107.3)
- C1, C10, C11, C12, C13, C14, C15, C16, C17, C2, C3, C4, C5, C6, C7, C8, C9: footprint Capacitor_SMD:C_0603_1608Metric -> Capacitor_SMD:C_0402_1005Metric-notxt
- D1, D10, D11, D12, D13, D14, D15, D16, D17, D18, D19, D2, D20, D21, D22, D23, D24, D25, D26, D27, D28, D29, D3, D30, D31, D32, D33, D34, D35, D36, D37, D38, D39, D4, D40, D41, D42, D43, D44, D45, D46, D47, D48, D49, D5, D50, D51, D52, D53, D54, D55, D56, D57, D58, D59, D6, D60, D61, D62, D63, D64, D7, D8, D9: footprint Diode_SMD:D_0603_1608Metric_NOTXTNOTFUCKD -> Diode_SMD:D_0603_1608Metric-notxt
- D100, D101, D102, D103, D104, D105, D106, D107, D108, D109, D110, D111, D112, D113, D114, D115, D116, D117, D118, D119, D120, D121, D122, D123, D124, D125, D126, D127, D128, D129, D130, D131, D132, D133, D134, D135, D136, D137, D138, D139, D140, D141, D142, D143, D144, D145, D146, D147, D148, D149, D150, D151, D152, D153, D154, D155, D156, D157, D158, D159, D160, D161, D162, D163, D164, D165, D166, D167, D168, D169, D170, D171, D172, D173, D174, D175, D176, D177, D178, D179, D180, D181, D182, D183, D184, D185, D186, D187, D188, D189, D190, D191, D192, D73, D74, D75, D76, D77, D78, D79, D80, D81, D82, D83, D84, D85, D86, D87, D88, D89, D90, D91, D92, D93, D94, D95, D96, D97, D98, D99: footprint LED_SMD:LED_WS2812B-2020_PLCC4_2.0x2.0mm -> LED_SMD:LED_WS2812B-2020_PLCC4_2.0x2.0mm-notext
- D193, D194, D195, D196, D197, D198, D199: value WS2812B-2020 -> D_Small; footprint LED_SMD:LED_WS2812B-2020_PLCC4_2.0x2.0mm -> Diode_SMD:D_0603_1608Metric-notxt; moved to B.Cu
- F1: footprint Fuse:Fuse_0603_1608Metric -> Fuse:Fuse_0402_1005Metric-notxt
- J1: footprint Connector_PinHeader_1.00mm:PinHeader_1x05_P1.00mm_Vertical_SMD_Pin1Right -> Connector_PinHeader_1.00mm:PinHeader_1x05_P1.00mm_Vertical_SMD_Pin1Right-notxt
- J2: footprint Connector_USB:USB_C_Receptacle_G-Switch_GT-USB-7025 -> Connector_USB:USB_C_Receptacle_G-Switch_GT-USB-7025-notxt
- MX1, MX10, MX11, MX12, MX13, MX14, MX15, MX16, MX17, MX18, MX19, MX2, MX20, MX21, MX22, MX23, MX24, MX25, MX26, MX27, MX28, MX29, MX3, MX30, MX31, MX32, MX33, MX34, MX35, MX36, MX37, MX38, MX39, MX4, MX40, MX41, MX42, MX43, MX44, MX45, MX46, MX47, MX48, MX49, MX5, MX50, MX51, MX52, MX53, MX54, MX55, MX56, MX57, MX58, MX59, MX6, MX60, MX61, MX62, MX63, MX64, MX7, MX8, MX9: footprint Arcade_Switch:OBSC-30 SW-68 -> Arcade_Switch:MM9-3-AU-withbutton
- R1, R2, R3, R4, R5, R6, R7: footprint Resistor_SMD:R_0603_1608Metric -> Resistor_SMD:R_0402_1005Metric-notext
- R8: footprint Resistor_SMD:R_0603_1608Metric -> Resistor_SMD:R_0402_1005Metric-notext; moved to B.Cu
- TP1: footprint TestPoint:TestPoint_Pad_4.0x4.0mm -> TestPoint:TestPoint_Pad_1.0x1.0mm-notxt
- U1: footprint Footprints:RP2040-QFN-56 -> Footprints:RP2040-QFN-56-notext
- U2: footprint W25Q16JVZPIQ:SON127P500X600X80-9N -> W25Q16JVZPIQ:SON127P500X600X80-9N-notxt
- U3: footprint Package_TO_SOT_SMD:SOT-23-6 -> Package_TO_SOT_SMD:SOT-23-6-notxt
- U4: footprint Package_TO_SOT_SMD:SOT-23-3 -> Package_TO_SOT_SMD:SOT-23-3-notxt
- Y1: footprint Crystal:Crystal_SMD_7050-4Pin_7.0x5.0mm -> Crystal:Crystal_SMD_2016-4Pin_2.0x1.6mm-notxt
- moved D73 362.6 mm to (-54.1, -296.2)
- moved D89 353.8 mm to (-54.1, -265.9)
- moved D105 345.8 mm to (-54.1, -235.6)
- moved D88 343.0 mm to (-68.3, -282.4), turned to 180 degrees
- moved D121 338.9 mm to (-54.1, -205.3)
- moved D74 334.5 mm to (-84.4, -296.2)
- moved D104 334.2 mm to (-68.3, -252.1), turned to 180 degrees
- moved D137 333.1 mm to (-54.1, -175.0)
- moved D153 327.7 mm to (-54.1, -144.7)
- moved D185 327.5 mm to (-54.1, -84.1)
- moved D169 327.0 mm to (-54.1, -114.4)
- moved D120 326.5 mm to (-68.3, -221.8), turned to 180 degrees
- moved D90 325.1 mm to (-84.4, -265.9)
- moved D136 319.8 mm to (-68.3, -191.5), turned to 180 degrees
- moved D106 316.6 mm to (-84.4, -235.6)
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Connections:
- D106 pad 3: Net-(D106-DIN) -> Net-(D105-DOUT)
- D107 pad 3: Net-(D105-DOUT) -> Net-(D106-DOUT)
- D107 pad 4: unconnected-(D107-VDD-Pad4) -> +5V
- D108 pad 1: Net-(D106-DIN) -> Net-(D108-DOUT)
- D108 pad 3: Net-(D108-DIN) -> Net-(D107-DOUT)
- D109 pad 2: unconnected-(D109-VSS-Pad2) -> GND
- D109 pad 3: Net-(D107-DOUT) -> Net-(D108-DOUT)
- D110 pad 1: Net-(D108-DIN) -> Net-(D110-DOUT)
- D110 pad 3: Net-(D110-DIN) -> Net-(D109-DOUT)
- D111 pad 3: Net-(D109-DOUT) -> Net-(D110-DOUT)
- D111 pad 4: unconnected-(D111-VDD-Pad4) -> +5V
- D112 pad 1: Net-(D110-DIN) -> Net-(D112-DOUT)
- D112 pad 3: Net-(D112-DIN) -> Net-(D111-DOUT)
- D113 pad 2: unconnected-(D113-VSS-Pad2) -> GND
- D113 pad 3: Net-(D111-DOUT) -> Net-(D112-DOUT)
- D114 pad 1: Net-(D112-DIN) -> Net-(D114-DOUT)
- D114 pad 3: Net-(D114-DIN) -> Net-(D113-DOUT)
- D115 pad 3: Net-(D113-DOUT) -> Net-(D114-DOUT)
- D115 pad 4: unconnected-(D115-VDD-Pad4) -> +5V
- D116 pad 1: Net-(D114-DIN) -> Net-(D116-DOUT)
- D116 pad 3: Net-(D116-DIN) -> Net-(D115-DOUT)
- D117 pad 2: unconnected-(D117-VSS-Pad2) -> GND
- D117 pad 3: Net-(D115-DOUT) -> Net-(D116-DOUT)
- D118 pad 1: Net-(D116-DIN) -> Net-(D118-DOUT)
- D118 pad 3: Net-(D118-DIN) -> Net-(D117-DOUT)
- D119 pad 3: Net-(D117-DOUT) -> Net-(D118-DOUT)
- D119 pad 4: unconnected-(D119-VDD-Pad4) -> +5V
- D120 pad 1: Net-(D118-DIN) -> Net-(D120-DOUT)
- D120 pad 3: Net-(D120-DIN) -> Net-(D119-DOUT)
- D121 pad 2: unconnected-(D121-VSS-Pad2) -> GND
- D121 pad 3: Net-(D119-DOUT) -> Net-(D120-DOUT)
- D122 pad 1: Net-(D120-DIN) -> Net-(D122-DOUT)
- D122 pad 3: Net-(D122-DIN) -> Net-(D121-DOUT)
- D123 pad 3: Net-(D121-DOUT) -> Net-(D122-DOUT)
- D123 pad 4: unconnected-(D123-VDD-Pad4) -> +5V
- D124 pad 1: Net-(D122-DIN) -> Net-(D124-DOUT)
- D124 pad 3: Net-(D124-DIN) -> Net-(D123-DOUT)
- D125 pad 2: unconnected-(D125-VSS-Pad2) -> GND
- D125 pad 3: Net-(D123-DOUT) -> Net-(D124-DOUT)
- D126 pad 1: Net-(D124-DIN) -> Net-(D126-DOUT)
- D126 pad 3: Net-(D126-DIN) -> Net-(D125-DOUT)
- D127 pad 3: Net-(D125-DOUT) -> Net-(D126-DOUT)
- D127 pad 4: unconnected-(D127-VDD-Pad4) -> +5V
- D128 pad 1: Net-(D126-DIN) -> Net-(D128-DOUT)
- D128 pad 3: Net-(D128-DIN) -> Net-(D127-DOUT)
- D129 pad 2: unconnected-(D129-VSS-Pad2) -> GND
- D129 pad 3: Net-(D127-DOUT) -> Net-(D128-DOUT)
- D130 pad 1: Net-(D128-DIN) -> Net-(D130-DOUT)
- D130 pad 3: Net-(D130-DIN) -> Net-(D129-DOUT)
- D131 pad 3: Net-(D129-DOUT) -> Net-(D130-DOUT)
- D131 pad 4: unconnected-(D131-VDD-Pad4) -> +5V
- D132 pad 1: Net-(D130-DIN) -> Net-(D132-DOUT)
- D132 pad 3: Net-(D132-DIN) -> Net-(D131-DOUT)
- D133 pad 2: unconnected-(D133-VSS-Pad2) -> GND
- D133 pad 3: Net-(D131-DOUT) -> Net-(D132-DOUT)
- D134 pad 1: Net-(D132-DIN) -> Net-(D134-DOUT)
- D134 pad 3: Net-(D134-DIN) -> Net-(D133-DOUT)
- D135 pad 3: Net-(D133-DOUT) -> Net-(D134-DOUT)
- D136 pad 1: Net-(D134-DIN) -> Net-(D136-DOUT)
- D137 pad 3: Net-(D106-DOUT) -> Net-(D136-DOUT)
- D138 pad 3: Net-(D138-DIN) -> Net-(D137-DOUT)
- D140 pad 1: unconnected-(D140-DOUT-Pad1) -> Net-(D140-DOUT)
- D140 pad 3: Net-(D140-DIN) -> Net-(D139-DOUT)
- D141 pad 3: Net-(D137-DOUT) -> Net-(D140-DOUT)
- D141 pad 4: unconnected-(D141-VDD-Pad4) -> +5V
- D142 pad 3: Net-(D139-DOUT) -> Net-(D141-DOUT)
- D142 pad 4: unconnected-(D142-VDD-Pad4) -> +5V
- D143 pad 1: Net-(D138-DIN) -> Net-(D143-DOUT)
- D143 pad 3: Net-(D143-DIN) -> Net-(D142-DOUT)
- D144 pad 1: Net-(D140-DIN) -> Net-(D144-DOUT)
- D144 pad 3: Net-(D144-DIN) -> Net-(D143-DOUT)
- D145 pad 2: unconnected-(D145-VSS-Pad2) -> GND
- D145 pad 3: Net-(D141-DOUT) -> Net-(D144-DOUT)
- D146 pad 2: unconnected-(D146-VSS-Pad2) -> GND
- D146 pad 3: Net-(D142-DOUT) -> Net-(D145-DOUT)
- D147 pad 1: Net-(D143-DIN) -> Net-(D147-DOUT)
- D147 pad 3: Net-(D147-DIN) -> Net-(D146-DOUT)
- D148 pad 1: Net-(D144-DIN) -> Net-(D148-DOUT)
- D148 pad 3: Net-(D148-DIN) -> Net-(D147-DOUT)
- D149 pad 3: Net-(D145-DOUT) -> Net-(D148-DOUT)
- D149 pad 4: unconnected-(D149-VDD-Pad4) -> +5V
- D150 pad 3: Net-(D146-DOUT) -> Net-(D149-DOUT)
- D150 pad 4: unconnected-(D150-VDD-Pad4) -> +5V
- D151 pad 1: Net-(D147-DIN) -> Net-(D151-DOUT)
- D151 pad 3: Net-(D151-DIN) -> Net-(D150-DOUT)
- D152 pad 1: Net-(D148-DIN) -> Net-(D152-DOUT)
- D152 pad 3: Net-(D152-DIN) -> Net-(D151-DOUT)
- D153 pad 2: unconnected-(D153-VSS-Pad2) -> GND
- D153 pad 3: Net-(D149-DOUT) -> Net-(D152-DOUT)
- D154 pad 2: unconnected-(D154-VSS-Pad2) -> GND
- D154 pad 3: Net-(D150-DOUT) -> Net-(D153-DOUT)
- D155 pad 1: Net-(D151-DIN) -> Net-(D155-DOUT)
- D155 pad 3: Net-(D155-DIN) -> Net-(D154-DOUT)
- D156 pad 1: Net-(D152-DIN) -> Net-(D156-DOUT)
- D156 pad 3: Net-(D156-DIN) -> Net-(D155-DOUT)
- D157 pad 3: Net-(D153-DOUT) -> Net-(D156-DOUT)
- D157 pad 4: unconnected-(D157-VDD-Pad4) -> +5V
- D158 pad 3: Net-(D154-DOUT) -> Net-(D157-DOUT)
- D158 pad 4: unconnected-(D158-VDD-Pad4) -> +5V
- D159 pad 1: Net-(D155-DIN) -> Net-(D159-DOUT)
- D159 pad 3: Net-(D159-DIN) -> Net-(D158-DOUT)
- D160 pad 1: Net-(D156-DIN) -> Net-(D160-DOUT)
- D160 pad 3: Net-(D160-DIN) -> Net-(D159-DOUT)
- D161 pad 2: unconnected-(D161-VSS-Pad2) -> GND
- D161 pad 3: Net-(D157-DOUT) -> Net-(D160-DOUT)
- D162 pad 2: unconnected-(D162-VSS-Pad2) -> GND
- D162 pad 3: Net-(D158-DOUT) -> Net-(D161-DOUT)
- D163 pad 1: Net-(D159-DIN) -> Net-(D163-DOUT)
- D163 pad 3: Net-(D163-DIN) -> Net-(D162-DOUT)
- D164 pad 1: Net-(D160-DIN) -> Net-(D164-DOUT)
- D164 pad 3: Net-(D164-DIN) -> Net-(D163-DOUT)
- D165 pad 3: Net-(D161-DOUT) -> Net-(D164-DOUT)
- D165 pad 4: unconnected-(D165-VDD-Pad4) -> +5V
- D166 pad 3: Net-(D162-DOUT) -> Net-(D165-DOUT)
- D166 pad 4: unconnected-(D166-VDD-Pad4) -> +5V
- D167 pad 1: Net-(D163-DIN) -> Net-(D167-DOUT)
- D167 pad 3: Net-(D167-DIN) -> Net-(D166-DOUT)
- D168 pad 1: Net-(D164-DIN) -> Net-(D168-DOUT)
- D168 pad 3: Net-(D168-DIN) -> Net-(D167-DOUT)
- D169 pad 2: unconnected-(D169-VSS-Pad2) -> GND
- D169 pad 3: Net-(D165-DOUT) -> Net-(D168-DOUT)
- D170 pad 2: unconnected-(D170-VSS-Pad2) -> GND
- D170 pad 3: Net-(D166-DOUT) -> Net-(D169-DOUT)
- D171 pad 1: Net-(D167-DIN) -> Net-(D171-DOUT)
- D171 pad 3: Net-(D171-DIN) -> Net-(D170-DOUT)
- D172 pad 1: Net-(D168-DIN) -> Net-(D172-DOUT)
- D172 pad 3: Net-(D172-DIN) -> Net-(D171-DOUT)
- D173 pad 3: Net-(D169-DOUT) -> Net-(D172-DOUT)
- D173 pad 4: unconnected-(D173-VDD-Pad4) -> +5V
- D174 pad 3: Net-(D170-DOUT) -> Net-(D173-DOUT)
- D174 pad 4: unconnected-(D174-VDD-Pad4) -> +5V
- D175 pad 1: Net-(D171-DIN) -> Net-(D175-DOUT)
- D175 pad 3: Net-(D175-DIN) -> Net-(D174-DOUT)
- D176 pad 1: Net-(D172-DIN) -> Net-(D176-DOUT)
- D176 pad 3: Net-(D176-DIN) -> Net-(D175-DOUT)
- D177 pad 2: unconnected-(D177-VSS-Pad2) -> GND
- D177 pad 3: Net-(D173-DOUT) -> Net-(D176-DOUT)
- D178 pad 2: unconnected-(D178-VSS-Pad2) -> GND
- D178 pad 3: Net-(D174-DOUT) -> Net-(D177-DOUT)
- D179 pad 1: Net-(D175-DIN) -> Net-(D179-DOUT)
- D179 pad 3: Net-(D179-DIN) -> Net-(D178-DOUT)
- D180 pad 1: Net-(D176-DIN) -> Net-(D180-DOUT)
- D180 pad 3: Net-(D180-DIN) -> Net-(D179-DOUT)
- D181 pad 3: Net-(D177-DOUT) -> Net-(D180-DOUT)
- D181 pad 4: unconnected-(D181-VDD-Pad4) -> +5V
- D182 pad 3: Net-(D178-DOUT) -> Net-(D181-DOUT)
- D182 pad 4: unconnected-(D182-VDD-Pad4) -> +5V
- D183 pad 1: Net-(D179-DIN) -> Net-(D183-DOUT)
- D183 pad 3: Net-(D183-DIN) -> Net-(D182-DOUT)
- D184 pad 1: Net-(D180-DIN) -> Net-(D184-DOUT)
- D184 pad 3: Net-(D184-DIN) -> Net-(D183-DOUT)
- D185 pad 2: unconnected-(D185-VSS-Pad2) -> GND
- D185 pad 3: Net-(D181-DOUT) -> Net-(D184-DOUT)
- D186 pad 2: unconnected-(D186-VSS-Pad2) -> GND
- D186 pad 3: Net-(D182-DOUT) -> Net-(D185-DOUT)
- D187 pad 1: Net-(D183-DIN) -> Net-(D187-DOUT)
- D187 pad 3: Net-(D187-DIN) -> Net-(D186-DOUT)
- D188 pad 1: Net-(D184-DIN) -> Net-(D188-DOUT)
- D188 pad 3: Net-(D188-DIN) -> Net-(D187-DOUT)
- D189 pad 3: Net-(D185-DOUT) -> Net-(D188-DOUT)
- D189 pad 4: unconnected-(D189-VDD-Pad4) -> +5V
- D190 pad 3: Net-(D186-DOUT) -> Net-(D189-DOUT)
- D190 pad 4: unconnected-(D190-VDD-Pad4) -> +5V
- D191 pad 1: Net-(D187-DIN) -> Net-(D191-DOUT)
- D191 pad 3: Net-(D191-DIN) -> Net-(D190-DOUT)
- D192 pad 1: Net-(D188-DIN) -> unconnected-(D192-DOUT-Pad1)
- D192 pad 3: Net-(D192-DIN) -> Net-(D191-DOUT)
- D193 pad 1: Net-(D193-DOUT) -> ROW0
- D193 pad 2: unconnected-(D193-VSS-Pad2) -> Net-(D193-A)
- D194 pad 1: Net-(D194-DOUT) -> ROW1
- D194 pad 2: unconnected-(D194-VSS-Pad2) -> Net-(D194-A)
- D195 pad 1: Net-(D191-DIN) -> ROW2
- D195 pad 2: GND -> Net-(D195-A)
- D196 pad 1: Net-(D192-DIN) -> ROW3
- D196 pad 2: GND -> Net-(D196-A)
- D197 pad 1: Net-(D197-DOUT) -> ROW4
- D197 pad 2: GND -> Net-(D197-A)
- D198 pad 1: Net-(D195-DIN) -> ROW5
- D198 pad 2: GND -> Net-(D198-A)
- D199 pad 1: Net-(D199-DOUT) -> ROW6
- D199 pad 2: GND -> Net-(D199-A)
- D73 pad 3: Net-(D73-DIN) -> Net-(D72-DOUT)
- D74 pad 4: unconnected-(D74-VDD-Pad4) -> +5V
- D75 pad 2: unconnected-(D75-VSS-Pad2) -> GND
- D76 pad 4: unconnected-(D76-VDD-Pad4) -> +5V
- D77 pad 2: unconnected-(D77-VSS-Pad2) -> GND
- D78 pad 4: unconnected-(D78-VDD-Pad4) -> +5V
- D79 pad 2: unconnected-(D79-VSS-Pad2) -> GND
- D80 pad 4: unconnected-(D80-VDD-Pad4) -> +5V
- D81 pad 2: unconnected-(D81-VSS-Pad2) -> GND
- D82 pad 4: unconnected-(D82-VDD-Pad4) -> +5V
- D83 pad 2: unconnected-(D83-VSS-Pad2) -> GND
- D84 pad 4: unconnected-(D84-VDD-Pad4) -> +5V
- D85 pad 2: unconnected-(D85-VSS-Pad2) -> GND
- D86 pad 4: unconnected-(D86-VDD-Pad4) -> +5V
- D87 pad 2: unconnected-(D87-VSS-Pad2) -> GND
- R8 pad 2: Net-(D73-DIN) -> Net-(D65-DIN)
- U1 pad 11: unconnected-(U1-GPIO8-Pad11) -> COL2
- U1 pad 12: unconnected-(U1-GPIO9-Pad12) -> COL1
- U1 pad 13: unconnected-(U1-GPIO10-Pad13) -> COL0
- U1 pad 14: unconnected-(U1-GPIO11-Pad14) -> COL8
- U1 pad 17: unconnected-(U1-GPIO14-Pad17) -> COL7
- U1 pad 18: unconnected-(U1-GPIO15-Pad18) -> COL6
- U1 pad 2: unconnected-(U1-GPIO0-Pad2) -> LED_DIN
- U1 pad 27: unconnected-(U1-GPIO16-Pad27) -> ROW0
- U1 pad 28: unconnected-(U1-GPIO17-Pad28) -> COL5
- U1 pad 3: unconnected-(U1-GPIO1-Pad3) -> ROW7
- U1 pad 34: unconnected-(U1-GPIO22-Pad34) -> COL4
- U1 pad 35: unconnected-(U1-GPIO23-Pad35) -> COL3
- U1 pad 4: unconnected-(U1-GPIO2-Pad4) -> ROW6
- U1 pad 5: unconnected-(U1-GPIO3-Pad5) -> ROW5
- U1 pad 6: unconnected-(U1-GPIO4-Pad6) -> ROW4
- U1 pad 7: unconnected-(U1-GPIO5-Pad7) -> ROW3
- U1 pad 8: unconnected-(U1-GPIO6-Pad8) -> ROW2
- U1 pad 9: unconnected-(U1-GPIO7-Pad9) -> ROW1
Routing:
- net GND: track 14.9 -> 4218.3 mm, vias 0 -> 177
- net +5V: track 21.4 -> 3079.6 mm, vias 2 -> 5
- net COL8: track 0.00 -> 358.2 mm, vias 0 -> 3
- net ROW7: track 212.1 -> 540.5 mm
- net ROW6: track 212.1 -> 512.0 mm
- net ROW5: track 212.1 -> 480.8 mm
- net ROW4: track 212.1 -> 449.6 mm
- net ROW3: track 212.1 -> 418.0 mm
- net ROW2: track 212.1 -> 383.4 mm
- net COL0: track 212.1 -> 364.3 mm, vias 0 -> 2
- net Net-(D65-DIN): track 0.00 -> 144.8 mm, vias 0 -> 1
- net ROW1: track 212.1 -> 356.3 mm
- net COL1: track 212.1 -> 332.5 mm, vias 0 -> 2
- net COL2: track 214.4 -> 300.3 mm, vias 0 -> 2
- net COL7: track 212.1 -> 292.2 mm, vias 0 -> 4
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- added copper zone on B.Cu, net COL8
