File: leds.kicad_sch (KiCad schematic)
At the start: 129 parts

Commit message: updates
Parts:
- removed D193, D194, D195, D196, D197, D198, D199, D200: WS2812B-2020, LED_SMD:LED_WS2812B-2020_PLCC4_2.0x2.0mm, symbol LED:WS2812B-2020
- added D81, D82, D83, D84, D85, D86, D87, D88: WS2812B-2020, LED_SMD:LED_WS2812B-2020_PLCC4_2.0x2.0mm-notext, symbol LED:WS2812B-2020
- D100, D101, D102, D103, D104, D105, D106, D107, D108, D109, D110, D111, D112, D113, D114, D115, D116, D117, D118, D119, D120, D121, D122, D123, D124, D125, D126, D127, D128, D129, D130, D131, D132, D133, D134, D135, D136, D137, D138, D139, D140, D141, D142, D143, D144, D145, D146, D147, D148, D149, D150, D151, D152, D153, D154, D155, D156, D157, D158, D159, D160, D161, D162, D163, D164, D165, D166, D167, D168, D169, D170, D171, D172, D173, D174, D175, D176, D177, D178, D179, D180, D181, D182, D183, D184, D185, D186, D187, D188, D189, D190, D191, D192, D89, D90, D91, D92, D93, D94, D95, D96, D97, D98, D99: footprint LED_SMD:LED_WS2812B-2020_PLCC4_2.0x2.0mm -> LED_SMD:LED_WS2812B-2020_PLCC4_2.0x2.0mm-notext
- D65: renamed from D73; footprint LED_SMD:LED_WS2812B-2020_PLCC4_2.0x2.0mm -> LED_SMD:LED_WS2812B-2020_PLCC4_2.0x2.0mm-notext
- D66: renamed from D74; footprint LED_SMD:LED_WS2812B-2020_PLCC4_2.0x2.0mm -> LED_SMD:LED_WS2812B-2020_PLCC4_2.0x2.0mm-notext
- D67: renamed from D75; footprint LED_SMD:LED_WS2812B-2020_PLCC4_2.0x2.0mm -> LED_SMD:LED_WS2812B-2020_PLCC4_2.0x2.0mm-notext
- D68: renamed from D76; footprint LED_SMD:LED_WS2812B-2020_PLCC4_2.0x2.0mm -> LED_SMD:LED_WS2812B-2020_PLCC4_2.0x2.0mm-notext
- D69: renamed from D77; footprint LED_SMD:LED_WS2812B-2020_PLCC4_2.0x2.0mm -> LED_SMD:LED_WS2812B-2020_PLCC4_2.0x2.0mm-notext
- D70: renamed from D78; footprint LED_SMD:LED_WS2812B-2020_PLCC4_2.0x2.0mm -> LED_SMD:LED_WS2812B-2020_PLCC4_2.0x2.0mm-notext
- D71: renamed from D79; footprint LED_SMD:LED_WS2812B-2020_PLCC4_2.0x2.0mm -> LED_SMD:LED_WS2812B-2020_PLCC4_2.0x2.0mm-notext
- D72: renamed from D80; footprint LED_SMD:LED_WS2812B-2020_PLCC4_2.0x2.0mm -> LED_SMD:LED_WS2812B-2020_PLCC4_2.0x2.0mm-notext
- D73: renamed from D81; footprint LED_SMD:LED_WS2812B-2020_PLCC4_2.0x2.0mm -> LED_SMD:LED_WS2812B-2020_PLCC4_2.0x2.0mm-notext
- D74: renamed from D82; footprint LED_SMD:LED_WS2812B-2020_PLCC4_2.0x2.0mm -> LED_SMD:LED_WS2812B-2020_PLCC4_2.0x2.0mm-notext
- D75: renamed from D83; footprint LED_SMD:LED_WS2812B-2020_PLCC4_2.0x2.0mm -> LED_SMD:LED_WS2812B-2020_PLCC4_2.0x2.0mm-notext
- D76: renamed from D84; footprint LED_SMD:LED_WS2812B-2020_PLCC4_2.0x2.0mm -> LED_SMD:LED_WS2812B-2020_PLCC4_2.0x2.0mm-notext
- D77: renamed from D85; footprint LED_SMD:LED_WS2812B-2020_PLCC4_2.0x2.0mm -> LED_SMD:LED_WS2812B-2020_PLCC4_2.0x2.0mm-notext
- D78: renamed from D86; footprint LED_SMD:LED_WS2812B-2020_PLCC4_2.0x2.0mm -> LED_SMD:LED_WS2812B-2020_PLCC4_2.0x2.0mm-notext
- D79: renamed from D87; footprint LED_SMD:LED_WS2812B-2020_PLCC4_2.0x2.0mm -> LED_SMD:LED_WS2812B-2020_PLCC4_2.0x2.0mm-notext
- D80: renamed from D88; footprint LED_SMD:LED_WS2812B-2020_PLCC4_2.0x2.0mm -> LED_SMD:LED_WS2812B-2020_PLCC4_2.0x2.0mm-notext
- R8: footprint Resistor_SMD:R_0603_1608Metric -> Resistor_SMD:R_0402_1005Metric-notext
Connections:
- net +5V: now also D107.4 (VDD), D111.4 (VDD), D123.4 (VDD), D127.4 (VDD), D131.4 (VDD), D141.4 (VDD), D142.4 (VDD), D149.4 (VDD), D150.4 (VDD), D157.4 (VDD), D158.4 (VDD), D165.4 (VDD), D166.4 (VDD), D173.4 (VDD), D174.4 (VDD), D181.4 (VDD), D182.4 (VDD), D189.4 (VDD), D190.4 (VDD), D66.4 (VDD), D68.4 (VDD), D70.4 (VDD), D72.4 (VDD), D74.4 (VDD), D76.4 (VDD), D78.4 (VDD), D81.4 (VDD), D82.4 (VDD), D83.4 (VDD), D84.4 (VDD), D85.4 (VDD), D86.4 (VDD), D87.4 (VDD), D88.4 (VDD)
- net GND: now also D117.2 (VSS), D121.2 (VSS), D125.2 (VSS), D129.2 (VSS), D133.2 (VSS), D145.2 (VSS), D146.2 (VSS), D153.2 (VSS), D154.2 (VSS), D161.2 (VSS), D162.2 (VSS), D169.2 (VSS), D170.2 (VSS), D177.2 (VSS), D178.2 (VSS), D185.2 (VSS), D186.2 (VSS), D67.2 (VSS), D69.2 (VSS), D71.2 (VSS), D73.2 (VSS), D75.2 (VSS), D77.2 (VSS), D79.2 (VSS), D81.2 (VSS), D82.2 (VSS), D83.2 (VSS), D84.2 (VSS), D85.2 (VSS), D86.2 (VSS), D87.2 (VSS), D88.2 (VSS)
- net at D134.3 (DIN): now also D133.1 (DOUT); no longer D136.1 (DOUT)
- net at D120.3 (DIN): now also D119.1 (DOUT); no longer D122.1 (DOUT)
- net at D122.3 (DIN): now also D121.1 (DOUT); no longer D124.1 (DOUT)
- net at D152.3 (DIN): now also D151.1 (DOUT); no longer D156.1 (DOUT)
- net at D156.3 (DIN): now also D155.1 (DOUT); no longer D160.1 (DOUT)
- net at D166.3 (DIN): now also D165.1 (DOUT); no longer D162.1 (DOUT)
- net at D158.1 (DOUT): now also D159.3 (DIN); no longer D162.3 (DIN)
- net at D118.1 (DOUT): now also D119.3 (DIN); no longer D116.3 (DIN)
- net at D120.1 (DOUT): now also D121.3 (DIN); no longer D118.3 (DIN)
- net at D175.3 (DIN): now also D174.1 (DOUT); no longer D179.1 (DOUT)
- net at D179.3 (DIN): now also D178.1 (DOUT); no longer D183.1 (DOUT)
- net at D117.1 (DOUT): now also D118.3 (DIN); no longer D119.3 (DIN)
- net at D80.1 (DOUT): now also D81.3 (DIN); no longer D89.3 (DIN)
- net at D153.1 (DOUT): now also D154.3 (DIN); no longer D157.3 (DIN)
- net at D153.3 (DIN): now also D152.1 (DOUT); no longer D149.1 (DOUT)
- net at D168.1 (DOUT): now also D169.3 (DIN); no longer D164.3 (DIN)
- net at D172.1 (DOUT): now also D173.3 (DIN); no longer D168.3 (DIN)
- net at D151.3 (DIN): now also D150.1 (DOUT); no longer D155.1 (DOUT)
- net at D155.3 (DIN): now also D154.1 (DOUT); no longer D159.1 (DOUT)
- net at D109.3 (DIN): now also D108.1 (DOUT); no longer D107.1 (DOUT)
- net at D107.3 (DIN): now also D106.1 (DOUT); no longer D105.1 (DOUT)
- net at D141.3 (DIN): now also D140.1 (DOUT); no longer D137.1 (DOUT)
- net at D137.3 (DIN): now also D136.1 (DOUT); no longer D106.1 (DOUT)
- net at D143.1 (DOUT): now also D144.3 (DIN); no longer D138.3 (DIN)
- net at D115.3 (DIN): now also D114.1 (DOUT); no longer D113.1 (DOUT)
- net at D113.3 (DIN): now also D112.1 (DOUT); no longer D111.1 (DOUT)
- net at D170.1 (DOUT): now also D171.3 (DIN); no longer D174.3 (DIN)
- net at D170.3 (DIN): now also D169.1 (DOUT); no longer D166.1 (DOUT)
- net at D134.1 (DOUT): now also D135.3 (DIN); no longer D132.3 (DIN)
- net at D126.1 (DOUT): now also D127.3 (DIN); no longer D124.3 (DIN)
- net at D140.3 (DIN): now also D139.1 (DOUT); no longer D144.1 (DOUT)
- net at D148.1 (DOUT): now also D149.3 (DIN); no longer D144.3 (DIN)
- net at D146.1 (DOUT): now also D147.3 (DIN); no longer D150.3 (DIN)
- net at D189.1 (DOUT): now also D190.3 (DIN)
- net at D185.1 (DOUT): now also D186.3 (DIN); no longer D189.3 (DIN)
- net at D106.3 (DIN): now also D105.1 (DOUT); no longer D108.1 (DOUT)
- net at D108.3 (DIN): now also D107.1 (DOUT); no longer D110.1 (DOUT)
- net at D126.3 (DIN): now also D125.1 (DOUT); no longer D128.1 (DOUT)
- net at D128.3 (DIN): now also D127.1 (DOUT); no longer D130.1 (DOUT)
- net at D161.3 (DIN): now also D160.1 (DOUT); no longer D157.1 (DOUT)
- net at D191.1 (DOUT): now also D192.3 (DIN); no longer D187.3 (DIN)
- net at D191.3 (DIN): now also D190.1 (DOUT)
- net at D185.3 (DIN): now also D184.1 (DOUT); no longer D181.1 (DOUT)
- net at D172.3 (DIN): now also D171.1 (DOUT); no longer D176.1 (DOUT)
- net at D133.3 (DIN): now also D132.1 (DOUT); no longer D131.1 (DOUT)
- net at D129.1 (DOUT): now also D130.3 (DIN); no longer D131.3 (DIN)
- net at D173.1 (DOUT): now also D174.3 (DIN); no longer D177.3 (DIN)
- net at D145.1 (DOUT): now also D146.3 (DIN); no longer D149.3 (DIN)
- net at D141.1 (DOUT): now also D142.3 (DIN); no longer D145.3 (DIN)
- net at D123.3 (DIN): now also D122.1 (DOUT); no longer D121.1 (DOUT)
- net at D142.1 (DOUT): now also D143.3 (DIN); no longer D146.3 (DIN)
- net at D158.3 (DIN): now also D157.1 (DOUT); no longer D154.1 (DOUT)
- net at D180.1 (DOUT): now also D181.3 (DIN); no longer D176.3 (DIN)
- net at D148.3 (DIN): now also D147.1 (DOUT); no longer D152.1 (DOUT)
- net at D184.3 (DIN): now also D183.1 (DOUT); no longer D188.1 (DOUT)
- net at D192.1 (DOUT): no longer D188.3 (DIN)
- net at D110.3 (DIN): now also D109.1 (DOUT); no longer D112.1 (DOUT)
- net at D112.3 (DIN): now also D111.1 (DOUT); no longer D114.1 (DOUT)
- net at D114.3 (DIN): now also D113.1 (DOUT); no longer D116.1 (DOUT)
- net at D180.3 (DIN): now also D179.1 (DOUT); no longer D184.1 (DOUT)
- net at D186.1 (DOUT): now also D187.3 (DIN); no longer D190.3 (DIN)
- net at D117.3 (DIN): now also D116.1 (DOUT); no longer D115.1 (DOUT)
- net at D125.3 (DIN): now also D124.1 (DOUT); no longer D123.1 (DOUT)
- net at D111.3 (DIN): now also D110.1 (DOUT); no longer D109.1 (DOUT)
- net at D129.3 (DIN): now also D128.1 (DOUT); no longer D127.1 (DOUT)
- net at D177.1 (DOUT): now also D178.3 (DIN); no longer D181.3 (DIN)
- net at D160.3 (DIN): now also D159.1 (DOUT); no longer D164.1 (DOUT)
- net at D182.1 (DOUT): now also D183.3 (DIN); no longer D186.3 (DIN)
- net at D182.3 (DIN): now also D181.1 (DOUT); no longer D178.1 (DOUT)
- net at D167.3 (DIN): now also D166.1 (DOUT); no longer D171.1 (DOUT)
- net at D175.1 (DOUT): now also D176.3 (DIN); no longer D171.3 (DIN)
- net at D163.1 (DOUT): now also D164.3 (DIN); no longer D159.3 (DIN)
- net at D167.1 (DOUT): now also D168.3 (DIN); no longer D163.3 (DIN)
- net at D165.3 (DIN): now also D164.1 (DOUT); no longer D161.1 (DOUT)
- net at D187.1 (DOUT): now also D188.3 (DIN); no longer D183.3 (DIN)
- new net: D83.1 (DOUT), D84.3 (DIN)
- new net: D82.1 (DOUT), D83.3 (DIN)
- new net: D86.1 (DOUT), D87.3 (DIN)
- new net: D85.1 (DOUT), D86.3 (DIN)
- new net: D87.1 (DOUT), D88.3 (DIN)
- new net: D84.1 (DOUT), D85.3 (DIN)
- new net: D137.1 (DOUT), D138.3 (DIN)
- new net: D81.1 (DOUT), D82.3 (DIN)
- new net: D149.1 (DOUT), D150.3 (DIN)
- new net: D144.1 (DOUT), D145.3 (DIN)
- new net: D131.1 (DOUT), D132.3 (DIN)
- new net: D130.1 (DOUT), D131.3 (DIN)
- new net: D188.1 (DOUT), D189.3 (DIN)
- new net: D156.1 (DOUT), D157.3 (DIN)
- new net: D162.1 (DOUT), D163.3 (DIN)
- new net: D88.1 (DOUT), D89.3 (DIN)
- new net: D176.1 (DOUT), D177.3 (DIN)
- new net: D123.1 (DOUT), D124.3 (DIN)
- new net: D161.1 (DOUT), D162.3 (DIN)
- new net: D115.1 (DOUT), D116.3 (DIN)
- no-connect marks 1 -> 2

Commit message: yeah have some updates my g
Parts:
- D100, D101, D102, D103, D104, D105, D106, D107, D108, D109, D110, D111, D112, D113, D114, D115, D116, D117, D118, D119, D120, D121, D122, D123, D124, D125, D126, D127, D128, D129, D130, D131, D132, D133, D134, D135, D136, D137, D138, D139, D140, D141, D142, D143, D144, D145, D146, D147, D148, D149, D150, D151, D152, D153, D154, D155, D156, D157, D158, D159, D160, D161, D162, D163, D164, D165, D166, D167, D168, D169, D170, D171, D172, D173, D174, D175, D176, D177, D178, D179, D180, D181, D182, D183, D184, D185, D186, D187, D188, D189, D190, D191, D192, D65, D66, D67, D68, D69, D70, D71, D72, D73, D74, D75, D76, D77, D78, D79, D80, D81, D82, D83, D84, D85, D86, D87, D88, D89, D90, D91, D92, D93, D94, D95, D96, D97, D98, D99: JLCPCB Part (none) -> C965555
- R8: JLCPCB Part (none) -> C124084
